File: Hardware_design_IoT/Interfaces.kicad_sch (KiCad schematic)
At the start: 7 parts, among them U6 TXB0104RGY

Commit message: Fin du projet
Parts:
- added C40, C51, C61: 100nF, Capacitor_SMD:C_0603_1608Metric_Pad1.08x0.95mm_HandSolder, symbol Device:C
- added C41: 10nF, Capacitor_SMD:C_0603_1608Metric_Pad1.08x0.95mm_HandSolder, symbol Device:C
- added C42, C53: 10pF, Capacitor_SMD:C_0603_1608Metric_Pad1.08x0.95mm_HandSolder, symbol Device:C
- added C43, C44, C45: 22pF, Capacitor_SMD:C_0603_1608Metric_Pad1.08x0.95mm_HandSolder, symbol Device:C
- added C52: 10uF, Capacitor_SMD:C_0603_1608Metric_Pad1.08x0.95mm_HandSolder, symbol Device:C
- added C54, C55, C56, C57: DNP, Capacitor_SMD:C_0402_1005Metric_Pad0.74x0.62mm_HandSolder, symbol Device:C
- added C58: 33nF, Capacitor_SMD:C_0402_1005Metric_Pad0.74x0.62mm_HandSolder, symbol Device:C
- added C59: 22pF, Capacitor_SMD:C_0402_1005Metric_Pad0.74x0.62mm_HandSolder, symbol Device:C
- added C60, C62: 4.7uF, Capacitor_SMD:C_0603_1608Metric_Pad1.08x0.95mm_HandSolder, symbol Device:C
- added D10, D11, D12, D6, D7, D8, D9: ESD9M5.0ST5G, ESD9M5.0ST5G:SODFL1060X40N, symbol ESD9M5.0ST5G:ESD9M5.0ST5G
- added D13, D16, D17: TVS, Diode_SMD:D_0603_1608Metric, symbol SparkFun-DiscreteSemi:D_TVS
- added D14: Green, LED_SMD:LED_0603_1608Metric, symbol SparkFun-LED:LED_Green_0603
- added D15: Red, LED_SMD:LED_0603_1608Metric, symbol SparkFun-LED:LED_Red_0603
- added J3: SMC-216, SMC-216:XUNPU_SMC-216, symbol SMC-216:SMC-216
- added J4, J9: UJ2-MIBH2-4-SMT, Micro_USB:CUI_UJ2-MIBH2-4-SMT, symbol Micro_USB:UJ2-MIBH2-4-SMT
- added J5: MEM2075-00-140-01-A, MEM2075-00-140-01-A:GCT_MEM2075-00-140-01-A, symbol MEM2075-00-140-01-A:MEM2075-00-140-01-A
- added J6, J7, J8: Conn_Coaxial, Connector_Coaxial:U.FL_Molex_MCRF_73412-0110_Vertical, symbol Connector:Conn_Coaxial
- added L2: 47nH, Inductor_SMD:L_0402_1005Metric, symbol Device:L
- added Q4, Q5: Q_NPN_BEC_BRT, Package_TO_SOT_SMD:SOT-23, symbol Device:Q_NPN_BEC_BRT
- added R24, R25, R26, R27: 22R, Resistor_SMD:R_0603_1608Metric, symbol Device:R
- added R28, R29: 2K, Resistor_SMD:R_0603_1608Metric, symbol Device:R
- added R30, R31: 22R, Resistor_SMD:R_0402_1005Metric, symbol Device:R
- added R32: 10R, Resistor_SMD:R_0402_1005Metric, symbol Device:R
- added R33: 10K, Resistor_SMD:R_0402_1005Metric, symbol Device:R
- added R34: 4.7K, Resistor_SMD:R_0402_1005Metric, symbol Device:R
- added U10: CP2102-GM, CP2102-GM:QFN50P500X500X100-29N, symbol CP2102-GM:CP2102-GM
- added U11, U7: USBLC6-2SC6, Package_TO_SOT_SMD:SOT-23-6, symbol Power_Protection:USBLC6-2SC6
- added U8: SMF05CT1G, SMF05CT1G:SOT65P210X110-6N, symbol SMF05CT1G:SMF05CT1G
Connections:
- net 3.3V: now also C60.2, C61.2, R32.2, R34.1, U10.6 (VDD), U10.7 (REGIN)
- net CP2102_TO_MODEM_RX: now also U10.26 (TXD)
- net CP2102_TO_MODEM_TX: now also U10.25 (RXD)
- net GND: now also C40.1, C41.1, C42.1, C43.1, C44.1, C45.1, C51.1, C52.1, C53.1, C54.1, C55.1, C56.1, C57.1, C58.2, C60.1, C61.1, C62.1, D10.2, D11.2, D12.2, D13.1 (A1), D16.1 (A1), D17.1 (A1), D6.2, D7.2, D8.2, D9.2, J3.C2 (GND), J3.S1 (SHIELD), J3.S2 (SHIELD), J4.5, J4.SH1 (SHIELD), J4.SH2 (SHIELD), J4.SH3 (SHIELD), J4.SH4 (SHIELD), J4.SH5 (SHIELD), J5.P6 (VSS), J5.SH1 (SHIELD), J5.SH2 (SHIELD), J5.SH3 (SHIELD), J5.SH4 (SHIELD), J6.2 (Ext), J7.2 (Ext), J8.2 (Ext), J9.5, J9.SH1 (SHIELD), J9.SH2 (SHIELD), J9.SH3 (SHIELD), J9.SH4 (SHIELD), J9.SH5 (SHIELD), Q4.2 (E), Q5.2 (E), R33.1, U10.29 (GND), U10.3 (GND), U11.2 (GND), U7.2 (GND), U8.2
- new net: C55.2, D13.2 (A2), J6.1 (In), R30.1
- new net: J3.C5 (CLK), R25.1, U8.4
- new net: C58.1, L2.1, R32.1
- new net: D15.1 (K), R28.1
- new net: J3.C3 (RST), R26.2, U8.6
- new net: J3.C6 (IO), R24.2, U8.5
- new net: C57.2, D16.2 (A2), J7.1 (In), R31.1
- new net: J4.2, U7.1 (I/O1)
- new net: J4.3, U7.3 (I/O2)
- new net: J4.1, U7.5 (VBUS)
- new net: J9.2, U11.1 (I/O1)
- new net: J9.3, U11.3 (I/O2)
- new net: U10.4 (D+), U11.4 (I/O2)
- new net: U10.5 (D–), U11.6 (I/O1)
- new net: Q4.3 (C), R28.2
- new net: C59.1, D17.2 (A2), J8.1 (In), L2.2
- new net: D6.1, J5.P5 (CLK), R27.1
- new net: D14.1 (K), R29.1
- new net: Q5.3 (C), R29.2
- new net: C62.2, U10.18 (NC/VPP)
- new net: R33.2, U10.11 (~{SUSPEND})
- new net: R34.2, U10.9 (~{RST})
- new net 3.V: C51.2, C52.2, C53.2, D7.1, J5.P4 (VDD)
- new net AUX_ANTENNA: C56.2, R31.2
- new net GNSS_ANTENNA: C59.2
- new net MAIN_ANTENNA: C54.2, R30.2
- new net NETLIGHT: Q4.1 (B)
- new net SD_CLK: R27.2
- new net SD_CMD: D8.1, J5.P3 (CMD)
- new net SD_DATA0: D9.1, J5.P7 (DAT0)
- new net SD_DATA1: D10.1, J5.P8 (DAT1)
- new net SD_DATA2: D11.1, J5.P1 (DAT2)
- new net SD_DATA3: D12.1, J5.P2 (CD/DAT3)
- new net SIM_CLK: C44.2, R25.2
- new net SIM_DATA: C45.2, R24.1
- new net SIM_RST: C43.2, R26.1
- new net SIM_VDD: C40.2, C41.2, C42.2, J3.C1 (VCC), U8.1
- new net STATUS: Q5.1 (B)
- new net USB_N: U7.6 (I/O1)
- new net USB_P: U7.4 (I/O2)
- new net VBUS: J9.1, U10.8 (VBUS), U11.5 (VBUS)
- new net VCC_LTEMODEM: D14.2 (A), D15.2 (A)
- no-connect marks 0 -> 12
Other:
- note added: "Auxilary Antenna"
- note added: "GNSS Antenna"
- note added: "GSM USB Interface Circuit"
- note added: "Main Antenna"
- note added: "Network and Status LEDs"
- note added: "SD Card Circuit"
- note added: "SD Card ESD Protection"
- note added: "SIM Card Circuit"
- note added: "SIM Card EMI Protection"
- note added: "SIM Card ESD Protection"
- note added: "USB ESD Protection"
- note added: "USB To UART Converter"
- moved on the sheet: C27, C39, R20, R21, R22, R23, U6
