File: Hardware_design_IoT/LTE_Modem_Unit.kicad_sch (KiCad schematic)
At the start: 6 parts, among them Q2 Q_NPN_BEC_BRT, Q3 Q_NPN_BEC_BRT, SW3 PWRKEY_SW, U5 SIM7600E-H

Commit message: Fin du projet
Parts:
- added DIP_RST2: DIP_RST, Button_Switch_SMD:SW_DIP_SPSTx01_Slide_6.7x4.1mm_W6.73mm_P2.54mm_LowProfile_JPin, symbol Switch:SW_DIP_x01
Connections:
- net 1.8V: now also DIP_RST2.1
- net USB_N: now reaches U5.12 (USB_DN)
- net USB_P: now reaches U5.13 (USB_DP)
- net SIM_DATA: now reaches U5.17 (USIM_DATA)
- net SIM_RST: now reaches U5.18 (USIM_RST)
- net SIM_CLK: now reaches U5.19 (USIM_CLK)
- net SIM_VDD: now reaches U5.20 (USIM_VDD)
- net SD_DATA1: now reaches U5.27 (SDIO_DATA1)
- net SD_DATA2: now reaches U5.28 (SDIO_DATA2)
- net SD_CMD: now reaches U5.29 (SDIO_CMD)
- net SD_DATA0: now reaches U5.30 (SDIO_DATA0)
- net SD_DATA3: now reaches U5.31 (SDIO_DATA3)
- net SD_CLK: now reaches U5.32 (SDIO_CLK)
- net STATUS: now reaches U5.49 (STATUS)
- net NETLIGHT: now reaches U5.51 (NETLIGHT)
- net AUX_ANTENNA: now reaches U5.59 (AUX_ANT)
- net GNSS_ANTENNA: now reaches U5.79 (GNSS_ANT)
- net MAIN_ANTENNA: now reaches U5.82 (MAIN_ANT)
- net at U5.85 (BOOT_CFG0): now also DIP_RST2.2
- no-connect marks 58 -> 40
Other:
- note added: "4G MODEM"
- moved on the sheet: C15, C26, Q2, Q3, SW3, U5
