File: Hardware_design_IoT/power_supply.kicad_sch (KiCad schematic)
At the start: 48 parts, among them J1 Barrel_Jack_Switch, Q1 Q_NPN_BEC_BRT, U1 MP1584EN, U2 TLV70033_SOT23-5, U4 LD39200DPUR

Commit message: Fin du projet
Parts:
- removed U1: MP1584EN, IoT_Library:SOIC127P600X170-9N, symbol IoT_Library:MP1584EN
- added C46, C49: 0.1uF, Capacitor_SMD:C_0603_1608Metric_Pad1.08x0.95mm_HandSolder, symbol SparkFun-Capacitor:C
- added C47, C48: 10uF, Capacitor_SMD:C_0603_1608Metric_Pad1.08x0.95mm_HandSolder, symbol SparkFun-Capacitor:C
- added C50: 22pF, Capacitor_SMD:C_0603_1608Metric_Pad1.08x0.95mm_HandSolder, symbol Device:C
- added FB4: FerriteBead, Ferrite_Bead:BEADC2012X105N, symbol Device:FerriteBead
- added U1: MP1584EN, MP1584EN:SOIC127P600X170-9N, symbol MP1584EN:MP1584EN
- added U9: LP5907MFX-3.0, Package_TO_SOT_SMD:SOT-23-5, symbol Regulator_Linear:LP5907MFX-3.0
Connections:
- net 5V: now also C46.1, C47.1, U9.1 (IN), U9.3 (EN)
- net GND: now also C46.2, C47.2, C48.2, C49.2, C50.2, U9.2 (GND)
- net GND-ISO: now also U1.5 (GND), U1.9 (GND)
- net at C1.1, C2.1, C3.1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: now also U1.7 (VIN)
- net at C4.1: now also U1.8 (BST)
- net at C4.2, D3.1 (K), L1.1: now also U1.1 (SW)
- net at R1.2, R2.1: now also U1.2 (EN)
- net at C5.1: now also U1.3 (COMP)
- net at R5.2, R6.1: now also U1.4 (FB)
- net at R3.1: now also U1.6 (FREQ)
- new net: C48.1, C49.1, C50.1, FB4.1, U9.5 (OUT)
- new net 3V: FB4.2
Other:
- note added: "Rating: 3V/250mA"
- note added: "SD Card LDO"
- moved on the sheet: C10, C11, C12, C13, C28, C29, C30, C31, C32, C33, C34, C35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
